File: Hardware/MPR121-Cap-Touch-Keypad.brd (EAGLE design)
At the start: 48.3 x 78.7 mm, 19 parts, among them IC1 MPR121

Commit message: Changing packages to Production IDs on caps/res
Parts:
- C1, C2: device SparkFun:0603-CAP -> SparkFun-Capacitors:0603-CAP
Changed lines of the file:
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@@
 <elements>
 <element name="IC1" library="SparkFun-Sensors" package="QFN-20-0.4MM-V2" value="MPR121" x="24.13" y="10.16" rot="MR90"/>
-<element name="C1" library="SparkFun" package="0603-CAP" value="0.1uF" x="13.97" y="6.985" rot="MR270"/>
+<element name="C1" library="SparkFun-Capacitors" package="0603-CAP" value="0.1uF" x="13.97" y="6.985" rot="MR270">
+<attribute name="PROD_ID" value="CAP-00810" x="13.97" y="6.985" size="1.778" layer="28" rot="MR270" display="off"/>
+<attribute name="VALUE" value="0.1uF" x="13.97" y="6.985" size="1.778" layer="28" rot="MR270" display="off"/>
+</element>
 <element name="R1" library="SparkFun" package="0603-RES" value="75k" x="11.43" y="6.985" rot="MR90"/>
-<element name="C2" library="SparkFun" package="0603-CAP" value="0.1uF" x="31.75" y="6.985" rot="MR90"/>
+<element name="C2" library="SparkFun-Capacitors" package="0603-CAP" value="0.1uF" x="31.75" y="6.985" rot="MR90">
+<attribute name="PROD_ID" value="CAP-00810" x="31.75" y="6.985" size="1.778" layer="28" rot="MR90" display="off"/>
+<attribute name="VALUE" value="0.1uF" x="31.75" y="6.985" size="1.778" layer="28" rot="MR90" display="off"/>
+</element>
 <element name="JP1" library="SparkFun" package="SFE-NEW-WEBLOGO" value="LOGO-SFENEW" x="33.655" y="39.751" rot="MR0"/>
 <element name="JP3" library="SparkFun" package="STAND-OFF" value="STAND-OFF" x="44.45" y="3.81" rot="MR0"/>
