File: Hardware/MPR121-Cap-Touch-Keypad.sch (EAGLE design)
At the start: 19 parts, among them IC1 MPR121

Commit message: Changing packages to Production IDs on caps/res
Parts:
- C1, C2: device SparkFun:CAP0603-CAP -> SparkFun-Capacitors:0.1UF-25V(+80/-20%)(0603)
Changed lines of the file:
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@@
 <part name="FRAME1" library="SparkFun-Aesthetics" deviceset="FRAME-LETTER" device=""/>
 <part name="IC1" library="SparkFun-Sensors" deviceset="MPR121" device="V2" value="MPR121"/>
-<part name="C1" library="SparkFun" deviceset="CAP" device="0603-CAP" value="0.1uF"/>
+<part name="C1" library="SparkFun-Capacitors" deviceset="0.1UF-25V(+80/-20%)(0603)" device="" value="0.1uF"/>
 <part name="GND1" library="SparkFun" deviceset="GND" device=""/>
 <part name="R1" library="SparkFun" deviceset="RESISTOR" device="0603-RES" value="75k"/>
@@
 <part name="GND4" library="SparkFun" deviceset="GND" device=""/>
 <part name="P+1" library="SparkFun" deviceset="VCC" device=""/>
-<part name="C2" library="SparkFun" deviceset="CAP" device="0603-CAP" value="0.1uF"/>
+<part name="C2" library="SparkFun-Capacitors" deviceset="0.1UF-25V(+80/-20%)(0603)" device="" value="0.1uF"/>
 <part name="P+2" library="SparkFun" deviceset="VCC" device=""/>
 <part name="GND5" library="SparkFun" deviceset="GND" device=""/>
